Commit message: Add verified Gazebo Harmonic simulation support
- gazebo.launch.py: gz-sim + spawn + controllers + ros_gz_bridge (config-file
  only: parameter_bridge ignores config_file when positional args are given,
  so /clock lives in the yaml). GZ_SIM_RESOURCE_PATH set for mesh URIs.
- worlds/rh8d_world.sdf selects bullet-featherstone: dartsim silently drops
  mimic constraints; bullet enforces them.
- World-anchored base with mass for gazebo (sdformat drops massless roots).
- gz joint-state-publisher plugin + bridge to /joint_states so mimic
  followers get TF in RViz during sim.
- Drive links got real virtual inertia: near-massless links broke actuation
  under featherstone.
- Sequential controller configs for both sides.
- E2E verified headless: mimic mode tracks perfectly (followers at exact
  ratios), fingertip wrench + palm IR topics publish; sequential mode
  documented as imperfect in current gz-physics (distal limit loses against
  stacked constraint) - see README.

Co-Authored-By: Claude Fable 5 <noreply@anthropic.com>

File: urdf/rh8d.gazebo.xacro (robot description, xacro)
@@ -37,4 +37,12 @@
   </xacro:macro>
   <xacro:macro name="rh8d_gazebo" params="prefix side">
+    <!-- Publishes ALL joint positions (including mimic followers, which are
+         not part of ros2_control) on <world>/model/<name>/joint_state; the
+         shipped bridge configs map it to /joint_states so RViz gets complete
+         TF during simulation. -->
+    <gazebo>
+      <plugin filename="gz-sim-joint-state-publisher-system"
+              name="gz::sim::systems::JointStatePublisher"/>
+    </gazebo>
     <xacro:rh8d_link_friction link="${prefix}forearm"/>
     <xacro:rh8d_link_friction link="${prefix}palm_axis"/>

File: urdf/rh8d.urdf.xacro (robot description, xacro)
@@ -21,5 +21,23 @@
   <xacro:property name="side"   value="$(arg side)"/>
   <xacro:property name="prefix" value="${'l_' if side == 'left' else 'r_'}"/>
-  <link name="base_link"/>
+  <!-- For Gazebo the model is anchored to the world and base_link needs mass,
+       otherwise sdformat drops the massless root and orphans the model. -->
+  <xacro:if value="$(arg use_gazebo)">
+    <link name="world"/>
+    <joint name="world_to_base" type="fixed">
+      <parent link="world"/>
+      <child link="base_link"/>
+    </joint>
+    <link name="base_link">
+      <inertial>
+        <origin rpy="0 0 0" xyz="0 0 0"/>
+        <mass value="0.05"/>
+        <inertia ixx="1e-05" ixy="0.0" ixz="0.0" iyy="1e-05" iyz="0.0" izz="1e-05"/>
+      </inertial>
+    </link>
+  </xacro:if>
+  <xacro:unless value="$(arg use_gazebo)">
+    <link name="base_link"/>
+  </xacro:unless>
   <xacro:rh8d prefix="${prefix}" side="${side}" parent="base_link"
               finger_coupling="$(arg finger_coupling)"

File: urdf/rh8d_finger.xacro (robot description, xacro)
@@ -94,9 +94,11 @@
        with staggered offsets so they engage one after another. -->
   <xacro:macro name="rh8d_drive_joint" params="prefix name parent upper">
+    <!-- Non-negligible virtual inertia: near-massless links destabilize the
+         featherstone solver and the mimic constraints anchored to this joint. -->
     <link name="${prefix}${name}_motor">
       <inertial>
         <origin rpy="0 0 0" xyz="0 0 0"/>
-        <mass value="1.0e-05"/>
-        <inertia ixx="1.0e-09" ixy="0.0" ixz="0.0" iyy="1.0e-09" iyz="0.0" izz="1.0e-09"/>
+        <mass value="0.01"/>
+        <inertia ixx="1.0e-06" ixy="0.0" ixz="0.0" iyy="1.0e-06" iyz="0.0" izz="1.0e-06"/>
       </inertial>
     </link>

Commit message: Fix contact explosion on object interaction
The Gazebo Classic/ODE contact params inherited from NICOL (mu 500,
kp 1e7, kd 1) made bullet-featherstone's impulse solver explode on the
very light finger links as soon as an object touched the hand: sustained
>18 rad/s joint velocities and limit violations. Replaced with realistic
values (mu 1.2 body / 1.5 rubber sensor pads, kp 1e5, kd 10).

Verified with a sphere spawned overlapping the closed fingers (worst
case): after the unavoidable interpenetration ejection transient the
grasp settles to <0.8 rad/s with limit violations at numerical-noise
level (0.001 rad).

Co-Authored-By: Claude Fable 5 <noreply@anthropic.com>

File: urdf/rh8d.gazebo.xacro (robot description, xacro)
@@ -4,10 +4,15 @@
        parameters, fingertip force_torque sensors and the palm IR distance
        sensor. Include via the rh8d_gazebo macro after instantiating rh8d. -->
-  <xacro:macro name="rh8d_link_friction" params="link">
+  <!-- Contact parameters. The original NICOL values (mu 500, kp 1e7, kd 1)
+       were tuned for Gazebo Classic/ODE and cause violent contact explosions
+       in bullet-featherstone (deep-penetration recovery on the very light
+       finger links); realistic friction and a soft, damped contact keep
+       grasping stable. -->
+  <xacro:macro name="rh8d_link_friction" params="link mu:=1.2">
     <gazebo reference="${link}">
-      <mu1>500.0</mu1>
-      <mu2>500.0</mu2>
-      <kp>10000000.0</kp>
-      <kd>1</kd>
+      <mu1>${mu}</mu1>
+      <mu2>${mu}</mu2>
+      <kp>100000.0</kp>
+      <kd>10.0</kd>
       <self_collide>1</self_collide>
     </gazebo>
@@ -29,5 +34,6 @@
       </sensor>
     </gazebo>
-    <xacro:rh8d_link_friction link="${prefix}${finger}_fingertip"/>
+    <!-- rubber sensor pads grip better than the plastic shells -->
+    <xacro:rh8d_link_friction link="${prefix}${finger}_fingertip" mu="1.5"/>
   </xacro:macro>
   <xacro:macro name="rh8d_finger_friction" params="prefix finger">
