Commit message: Move Gazebo sim to dartsim; bullet only for experimental sequential mode
bullet-featherstone has a severe runtime-insertion bug: adding any model to
a running world (a sphere from the GUI, 0.5 m away, zero contact) makes the
existing hand articulation thrash at 100 rad/s indefinitely. Reproduced and
verified; dartsim is unaffected.

- worlds/rh8d_world.sdf is now dartsim (default for mimic/independent);
  bullet lives on in rh8d_world_bullet.sdf, used only by sequential mode
  (its offset constraints exist nowhere else), documented as experimental.
- mimic mode works on dartsim by declaring the follower joints in the
  ros2_control block (state-only): ros2_control picks up the URDF <mimic>
  tags and gz_ros2_control enforces the coupling (offsets are all zero in
  this mode, so its offset bug is irrelevant). Verified: exact ratios.
- Verified on dartsim: far-sphere insertion (hand unaffected, 0.07 rad/s),
  overlapping-sphere spawn (no reaction), grasp closing capped at the
  2 rad/s joint velocity limit (dartsim enforces it; bullet did not),
  zero limit violations throughout.

Co-Authored-By: Claude Fable 5 <noreply@anthropic.com>

File: urdf/rh8d.ros2_control.xacro (robot description, xacro)
@@ -14,4 +14,16 @@
     <joint name="${joint}">
       <command_interface name="position"/>
+      <state_interface name="position"/>
+      <state_interface name="velocity"/>
+      <state_interface name="effort"/>
+    </joint>
+  </xacro:macro>
+  <!-- Mimic follower: state only. ros2_control picks up the URDF <mimic> tag
+       and gz_ros2_control enforces the coupling in simulation - this is what
+       makes 'mimic' mode work on dartsim, which drops SDF mimic constraints.
+       (Offsets are ignored by gz_ros2_control, but 'mimic' mode only uses
+       offset 0 so that is harmless here.) -->
+  <xacro:macro name="rh8d_follower_iface" params="joint">
+    <joint name="${joint}">
       <state_interface name="position"/>
       <state_interface name="velocity"/>
@@ -45,4 +57,17 @@
           <xacro:rh8d_joint_iface joint="${prefix}little_proximal_joint"/>
         </xacro:unless>
+        <xacro:rh8d_follower_iface joint="${prefix}thumb_medial_joint"/>
+        <xacro:rh8d_follower_iface joint="${prefix}thumb_distal_joint"/>
+        <xacro:rh8d_follower_iface joint="${prefix}index_medial_joint"/>
+        <xacro:rh8d_follower_iface joint="${prefix}index_distal_joint"/>
+        <xacro:rh8d_follower_iface joint="${prefix}middle_medial_joint"/>
+        <xacro:rh8d_follower_iface joint="${prefix}middle_distal_joint"/>
+        <xacro:rh8d_follower_iface joint="${prefix}ring_medial_joint"/>
+        <xacro:rh8d_follower_iface joint="${prefix}ring_distal_joint"/>
+        <xacro:rh8d_follower_iface joint="${prefix}little_medial_joint"/>
+        <xacro:rh8d_follower_iface joint="${prefix}little_distal_joint"/>
+        <xacro:if value="${couple}">
+          <xacro:rh8d_follower_iface joint="${prefix}little_proximal_joint"/>
+        </xacro:if>
       </xacro:if>
       <xacro:if value="${finger_coupling == 'sequential'}">

Commit message: Remove sequential coupling mode
The staggered-mimic-offset mechanism only ever worked in engines with
native offset constraints, and the sole such engine in Gazebo
(bullet-featherstone) is too unstable to ship. The coupling controller in
independent mode provides the same sequential closing with correct limits
plus adaptive wrap, on dartsim.

- xacros: drive-joint macro and all sequential branches removed; modes are
  now mimic | independent
- deleted: bullet world, sequential controller yamls, mimic_joint_clamper
  (only needed to visualize offset clamping in RViz)
- the motor slider GUI no longer borrows the sequential variant's
  description: rh8d_coupling_node generates a minimal motor-panel URDF
  (one revolute joint per motor axis) and latches it on motor_description
- launches/tests/README updated; committed plain URDFs verified unchanged;
  coupling behavior re-verified in Gazebo after the removal

Co-Authored-By: Claude Fable 5 <noreply@anthropic.com>

File: urdf/rh8d.ros2_control.xacro (robot description, xacro)
@@ -4,7 +4,5 @@
     ros2_control description for the RH8D.
     Only the joints that correspond to real actuators get command interfaces;
-    mimic followers are resolved by the simulator (or by the hand firmware on
-    real hardware) and are intentionally NOT listed here, so gz_ros2_control
-    never touches them.
+    mimic followers are declared with state interfaces only (see below).
     hardware_plugin: plugin for real hardware; defaults to mock components so
                      the description works out of the box. Replace with the
@@ -71,16 +69,4 @@
         </xacro:if>
       </xacro:if>
-      <xacro:if value="${finger_coupling == 'sequential'}">
-        <xacro:rh8d_joint_iface joint="${prefix}thumb_flexion_joint"/>
-        <xacro:rh8d_joint_iface joint="${prefix}index_flexion_joint"/>
-        <xacro:rh8d_joint_iface joint="${prefix}middle_flexion_joint"/>
-        <xacro:if value="${couple}">
-          <xacro:rh8d_joint_iface joint="${prefix}ring_little_flexion_joint"/>
-        </xacro:if>
-        <xacro:unless value="${couple}">
-          <xacro:rh8d_joint_iface joint="${prefix}ring_flexion_joint"/>
-          <xacro:rh8d_joint_iface joint="${prefix}little_flexion_joint"/>
-        </xacro:unless>
-      </xacro:if>
       <xacro:if value="${finger_coupling == 'independent'}">
         <xacro:rh8d_joint_iface joint="${prefix}thumb_proximal_joint"/>

File: urdf/rh8d.urdf.xacro (robot description, xacro)
@@ -3,5 +3,5 @@
   <!--
     Standalone RH8D hand.
-      xacro rh8d.urdf.xacro side:=left finger_coupling:=mimic
+      xacro rh8d.urdf.xacro side:=left finger_coupling:=mimic|independent
     To mount the hand on a robot, include rh8d_macro.xacro (and optionally
     rh8d.gazebo.xacro / rh8d.ros2_control.xacro) and instantiate the macros

File: urdf/rh8d_finger.xacro (robot description, xacro)
@@ -90,36 +90,11 @@
     </link>
   </xacro:macro>
-  <!-- Virtual motor joint used in 'sequential' coupling mode. Represents the
-       actuator position of one flexion tendon; the phalanx joints mimic it
-       with staggered offsets so they engage one after another. -->
-  <xacro:macro name="rh8d_drive_joint" params="prefix name parent upper">
-    <!-- Non-negligible virtual inertia: near-massless links destabilize the
-         featherstone solver and the mimic constraints anchored to this joint. -->
-    <link name="${prefix}${name}_motor">
-      <inertial>
-        <origin rpy="0 0 0" xyz="0 0 0"/>
-        <mass value="0.01"/>
-        <inertia ixx="1.0e-06" ixy="0.0" ixz="0.0" iyy="1.0e-06" iyz="0.0" izz="1.0e-06"/>
-      </inertial>
-    </link>
-    <joint name="${prefix}${name}_joint" type="revolute">
-      <origin rpy="0 0 0" xyz="0 0 0"/>
-      <parent link="${parent}"/>
-      <child link="${prefix}${name}_motor"/>
-      <axis xyz="0 0 1"/>
-      <limit effort="20" lower="0.0" upper="${upper}" velocity="2"/>
-      <dynamics damping="0.1" friction="0.0"/>
-    </joint>
-  </xacro:macro>
   <!--
     One finger (index/middle/ring/little): proximal, medial, distal phalanges
     plus the fingertip sensor pad.
-    coupling: 'mimic' | 'sequential' | 'independent'
-    leader:   name of the joint the finger follows.
-              mimic:      ''            -> proximal is the leader (own motor);
-                          '<joint>'     -> whole finger follows that joint
-                                           (little finger following the ring
-                                           proximal joint on the real hand)
-              sequential: '<drive joint>' (required)
+    coupling: 'mimic' | 'independent'
+    leader:   mimic mode only: '' -> proximal is the leader (own motor);
+              '<joint>' -> whole finger follows that joint (little finger
+              following the ring proximal joint on the real hand)
     mount_*:  palm mount origin, already side-mirrored by the caller.
   -->
@@ -134,7 +109,4 @@
       <limit effort="20" lower="0.0" upper="${finger_prox_upper}" velocity="2"/>
       <dynamics damping="0.02" friction="0.0"/>
-      <xacro:if value="${coupling == 'sequential'}">
-        <mimic joint="${leader}" multiplier="1.0" offset="0.0"/>
-      </xacro:if>
       <xacro:if value="${coupling == 'mimic' and leader != ''}">
         <mimic joint="${leader}" multiplier="1.0" offset="0.0"/>
@@ -151,7 +123,4 @@
       <limit effort="20" lower="0.0" upper="${finger_med_upper}" velocity="2"/>
       <dynamics damping="0.01" friction="0.0"/>
-      <xacro:if value="${coupling == 'sequential'}">
-        <mimic joint="${leader}" multiplier="1.0" offset="${-finger_prox_upper}"/>
-      </xacro:if>
       <xacro:if value="${coupling == 'mimic'}">
         <mimic joint="${mimic_base}" multiplier="${finger_med_mult}" offset="0.0"/>
@@ -168,7 +137,4 @@
       <limit effort="20" lower="0.0" upper="${finger_dist_upper}" velocity="2"/>
       <dynamics damping="0.001" friction="0.0"/>
-      <xacro:if value="${coupling == 'sequential'}">
-        <mimic joint="${leader}" multiplier="1.0" offset="${-(finger_prox_upper + finger_med_upper)}"/>
-      </xacro:if>
       <xacro:if value="${coupling == 'mimic'}">
         <mimic joint="${mimic_base}" multiplier="${finger_dist_mult}" offset="0.0"/>
@@ -219,7 +185,4 @@
       <limit effort="20" lower="0.0" upper="${thumb_prox_upper}" velocity="2"/>
       <dynamics damping="0.01" friction="0.0"/>
-      <xacro:if value="${coupling == 'sequential'}">
-        <mimic joint="${leader}" multiplier="1.0" offset="0.0"/>
-      </xacro:if>
     </joint>
     <link name="${prefix}thumb_proximal">
@@ -244,7 +207,4 @@
       <limit effort="20" lower="0.0" upper="${thumb_med_upper}" velocity="2"/>
       <dynamics damping="0.01" friction="0.0"/>
-      <xacro:if value="${coupling == 'sequential'}">
-        <mimic joint="${leader}" multiplier="1.0" offset="${-thumb_prox_upper}"/>
-      </xacro:if>
       <xacro:if value="${coupling == 'mimic'}">
         <mimic joint="${mimic_base}" multiplier="${thumb_med_mult}" offset="0.0"/>
@@ -284,7 +244,4 @@
       <limit effort="20" lower="0.0" upper="${thumb_dist_upper}" velocity="2"/>
       <dynamics damping="0.001" friction="0.0"/>
-      <xacro:if value="${coupling == 'sequential'}">
-        <mimic joint="${leader}" multiplier="1.0" offset="${-(thumb_prox_upper + thumb_med_upper)}"/>
-      </xacro:if>
       <xacro:if value="${coupling == 'mimic'}">
         <mimic joint="${mimic_base}" multiplier="${thumb_dist_mult}" offset="0.0"/>

File: urdf/rh8d_macro.xacro (robot description, xacro)
@@ -12,11 +12,7 @@
                                         linearly (8-DOF interface, safe with all
                                         standard tools)
-                        'sequential'  - virtual motor joint per flexion tendon;
-                                        phalanges engage one after another via
-                                        staggered mimic offsets clamped by their
-                                        joint limits (physics engines only; use
-                                        the shipped mimic_joint_clamper for RViz)
-                        'independent' - every phalanx joint actuated (21-DOF,
-                                        NICOL-style, for tendon research)
+                        'independent' - every phalanx joint actuated; combine
+                                        with rh8d_coupling_node.py for
+                                        tendon-like sequential/adaptive closing
     couple_ring_little: ring and little finger share one actuator (matches the
                         real hand); ignored in 'independent' mode
@@ -24,5 +20,4 @@
   <xacro:macro name="rh8d" params="prefix side parent *origin finger_coupling:=mimic couple_ring_little:=true">
     <xacro:property name="reflect" value="${1 if side == 'left' else -1}"/>
-    <xacro:property name="seq"     value="${finger_coupling == 'sequential'}"/>
     <xacro:property name="couple"  value="${couple_ring_little in [True, 'true', 'True', '1', 1]}"/>
     <!-- ======================= wrist chain ======================= -->
@@ -131,35 +126,10 @@
       </inertial>
     </link>
-    <!-- ================== flexion drive actuators ================== -->
-    <!-- Virtual motor joints exist only in 'sequential' mode; they carry the
-         one-command-per-tendon interface that matches the real actuators. -->
-    <xacro:if value="${seq}">
-      <xacro:rh8d_drive_joint prefix="${prefix}" name="thumb_flexion" parent="${prefix}palm"
-                              upper="${0.8 + 1.57 + 0.4}"/>
-      <xacro:rh8d_drive_joint prefix="${prefix}" name="index_flexion" parent="${prefix}palm"
-                              upper="${1.57 + 1.57 + 1.0}"/>
-      <xacro:rh8d_drive_joint prefix="${prefix}" name="middle_flexion" parent="${prefix}palm"
-                              upper="${1.57 + 1.57 + 1.0}"/>
-      <xacro:if value="${couple}">
-        <xacro:rh8d_drive_joint prefix="${prefix}" name="ring_little_flexion" parent="${prefix}palm"
-                                upper="${1.57 + 1.57 + 1.0}"/>
-      </xacro:if>
-      <xacro:unless value="${couple}">
-        <xacro:rh8d_drive_joint prefix="${prefix}" name="ring_flexion" parent="${prefix}palm"
-                                upper="${1.57 + 1.57 + 1.0}"/>
-        <xacro:rh8d_drive_joint prefix="${prefix}" name="little_flexion" parent="${prefix}palm"
-                                upper="${1.57 + 1.57 + 1.0}"/>
-      </xacro:unless>
-    </xacro:if>
-    <xacro:property name="ring_leader"
-        value="${(prefix + ('ring_little_flexion_joint' if couple else 'ring_flexion_joint')) if seq else ''}"/>
     <xacro:property name="little_leader"
-        value="${(prefix + ('ring_little_flexion_joint' if couple else 'little_flexion_joint')) if seq
-                 else (prefix + 'ring_proximal_joint' if (couple and finger_coupling == 'mimic') else '')}"/>
+        value="${prefix + 'ring_proximal_joint' if (couple and finger_coupling == 'mimic') else ''}"/>
     <!-- ======================= thumb ======================= -->
     <!-- The thumb abduction mount is calibrated per side (not an exact mirror). -->
     <xacro:if value="${side == 'left'}">
       <xacro:rh8d_thumb prefix="${prefix}" coupling="${finger_coupling}"
-                        leader="${prefix + 'thumb_flexion_joint' if seq else ''}"
                         mount_xyz="-0.0083412575 0.0157859987 -0.0379541955"
                         mount_rpy="0.60093862 -0.59510795 -2.8183247"
@@ -168,5 +138,4 @@
     <xacro:if value="${side == 'right'}">
       <xacro:rh8d_thumb prefix="${prefix}" coupling="${finger_coupling}"
-                        leader="${prefix + 'thumb_flexion_joint' if seq else ''}"
                         mount_xyz="-0.0083412575 0.0157859987 0.0379541955"
                         mount_rpy="-2.54680616 -0.60124514 0.33418237"
@@ -175,13 +144,10 @@
     <!-- ======================= fingers ======================= -->
     <xacro:rh8d_finger prefix="${prefix}" finger="index" coupling="${finger_coupling}"
-                       leader="${prefix + 'index_flexion_joint' if seq else ''}"
                        mount_xyz="-0.0043044918 0.0812907302 ${-0.0367863551*reflect}"
                        mount_rpy="${0.08267713*reflect} ${-0.17715231*reflect} -2.93857995"/>
     <xacro:rh8d_finger prefix="${prefix}" finger="middle" coupling="${finger_coupling}"
-                       leader="${prefix + 'middle_flexion_joint' if seq else ''}"
                        mount_xyz="-0.0012008743 0.0828960623 ${-0.0118294206*reflect}"
                        mount_rpy="${0.02*reflect} ${-0.06*reflect} -2.92246721"/>
     <xacro:rh8d_finger prefix="${prefix}" finger="ring" coupling="${finger_coupling}"
-                       leader="${ring_leader}"
                        mount_xyz="-0.0011171786 0.0818708881 ${0.0130285291*reflect}"
                        mount_rpy="${-0.06*reflect} ${0.04*reflect} -2.92922802"/>
