Commit message: Tune actuators and fix dartsim frozen-joint bug at limit rest poses
Snappier control (user request): phalanx effort 20->30, velocity 2->4;
wrist adduction/flexion effort 20->30, velocity 2->3, damping 5->1;
wrist rotation effort 0.5->10, velocity 1->3; thumb abduction damping
0.3->0.1. Centralized as xacro properties (phalanx_effort/velocity/lower).

Frozen thumb fix: joints whose rest pose sits exactly ON a position limit
are pinned by dartsim's limit constraint and never move - neither commands
(10x gain), gravity, nor disabling self-collision freed them; only being
knocked off the limit by other motion did (the reported 'thumb only moves
after wrist jiggle'). All flexion joints had lower=0.0 = spawn pose. Lower
limits are now -0.05 rad (matches the real tendon fingers' slack), keeping
the rest pose strictly inside the range.

Verified: thumb reaches 90% of a flexion step in 1.55s from cold start,
index full sequential close in 1.6s at peak 3.58 rad/s.

Co-Authored-By: Claude Fable 5 <noreply@anthropic.com>

File: urdf/rh8d_finger.xacro (robot description, xacro)
@@ -10,4 +10,14 @@
   <xacro:property name="finger_med_mult"   value="${finger_med_upper / finger_prox_upper}"/>
   <xacro:property name="finger_dist_mult"  value="${finger_dist_upper / finger_prox_upper}"/>
+  <!-- Actuator strength/speed (tuned up from the sluggish NICOL originals:
+       effort 20 / velocity 2 left the fingers slow and the thumb prone to
+       sticking against the palm until jostled). -->
+  <xacro:property name="phalanx_effort"    value="30"/>
+  <xacro:property name="phalanx_velocity"  value="4"/>
+  <!-- Slightly negative lower limit: joints parked exactly ON a limit get
+       pinned by dartsim's limit constraint and never move (frozen-thumb bug);
+       a few degrees of backward slack matches the real tendon fingers and
+       keeps the rest pose strictly inside the range. -->
+  <xacro:property name="phalanx_lower"     value="-0.05"/>
   <xacro:macro name="rh8d_phalanx_link" params="name mass com_y ixx iyy izz cyl_len cyl_rad cyl_y sph_y">
     <link name="${name}">
@@ -107,5 +117,5 @@
       <child link="${prefix}${finger}_proximal"/>
       <axis xyz="0 0 1"/>
-      <limit effort="20" lower="0.0" upper="${finger_prox_upper}" velocity="2"/>
+      <limit effort="${phalanx_effort}" lower="${phalanx_lower}" upper="${finger_prox_upper}" velocity="${phalanx_velocity}"/>
       <dynamics damping="0.02" friction="0.0"/>
       <xacro:if value="${coupling == 'mimic' and leader != ''}">
@@ -121,5 +131,5 @@
       <child link="${prefix}${finger}_medial"/>
       <axis xyz="0 0 1"/>
-      <limit effort="20" lower="0.0" upper="${finger_med_upper}" velocity="2"/>
+      <limit effort="${phalanx_effort}" lower="${phalanx_lower}" upper="${finger_med_upper}" velocity="${phalanx_velocity}"/>
       <dynamics damping="0.01" friction="0.0"/>
       <xacro:if value="${coupling == 'mimic'}">
@@ -135,5 +145,5 @@
       <child link="${prefix}${finger}_distal"/>
       <axis xyz="0 0 1"/>
-      <limit effort="20" lower="0.0" upper="${finger_dist_upper}" velocity="2"/>
+      <limit effort="${phalanx_effort}" lower="${phalanx_lower}" upper="${finger_dist_upper}" velocity="${phalanx_velocity}"/>
       <dynamics damping="0.001" friction="0.0"/>
       <xacro:if value="${coupling == 'mimic'}">
@@ -161,6 +171,6 @@
       <child link="${prefix}thumb_base"/>
       <axis xyz="${mount_axis}"/>
-      <limit effort="20" lower="-0.6" upper="${pi/4}" velocity="2"/>
-      <dynamics damping="0.3" friction="0.0"/>
+      <limit effort="${phalanx_effort}" lower="-0.6" upper="${pi/4}" velocity="${phalanx_velocity}"/>
+      <dynamics damping="0.1" friction="0.0"/>
     </joint>
     <link name="${prefix}thumb_base">
@@ -183,5 +193,5 @@
       <child link="${prefix}thumb_proximal"/>
       <axis xyz="0 0 1"/>
-      <limit effort="20" lower="0.0" upper="${thumb_prox_upper}" velocity="2"/>
+      <limit effort="${phalanx_effort}" lower="${phalanx_lower}" upper="${thumb_prox_upper}" velocity="${phalanx_velocity}"/>
       <dynamics damping="0.01" friction="0.0"/>
     </joint>
@@ -205,5 +215,5 @@
       <child link="${prefix}thumb_medial"/>
       <axis xyz="0 0 1"/>
-      <limit effort="20" lower="0.0" upper="${thumb_med_upper}" velocity="2"/>
+      <limit effort="${phalanx_effort}" lower="${phalanx_lower}" upper="${thumb_med_upper}" velocity="${phalanx_velocity}"/>
       <dynamics damping="0.01" friction="0.0"/>
       <xacro:if value="${coupling == 'mimic'}">
@@ -242,5 +252,5 @@
       <child link="${prefix}thumb_distal"/>
       <axis xyz="0 0 1"/>
-      <limit effort="20" lower="0.0" upper="${thumb_dist_upper}" velocity="2"/>
+      <limit effort="${phalanx_effort}" lower="${phalanx_lower}" upper="${thumb_dist_upper}" velocity="${phalanx_velocity}"/>
       <dynamics damping="0.001" friction="0.0"/>
       <xacro:if value="${coupling == 'mimic'}">

File: urdf/rh8d_left.urdf (robot description, URDF)
Before this commit: robot rh8d, 27 links, 26 joints
Joints:
- joint l_index_distal_joint: limit lower=0.0 upper=1.0 effort=20 velocity=2 -> lower=-0.05 upper=1.0 effort=30 velocity=4
- joint l_index_medial_joint: limit lower=0.0 upper=1.57 effort=20 velocity=2 -> lower=-0.05 upper=1.57 effort=30 velocity=4
- joint l_index_proximal_joint: limit lower=0.0 upper=1.57 effort=20 velocity=2 -> lower=-0.05 upper=1.57 effort=30 velocity=4
- joint l_little_distal_joint: limit lower=0.0 upper=1.0 effort=20 velocity=2 -> lower=-0.05 upper=1.0 effort=30 velocity=4
- joint l_little_medial_joint: limit lower=0.0 upper=1.57 effort=20 velocity=2 -> lower=-0.05 upper=1.57 effort=30 velocity=4
- joint l_little_proximal_joint: limit lower=0.0 upper=1.57 effort=20 velocity=2 -> lower=-0.05 upper=1.57 effort=30 velocity=4
- joint l_middle_distal_joint: limit lower=0.0 upper=1.0 effort=20 velocity=2 -> lower=-0.05 upper=1.0 effort=30 velocity=4
- joint l_middle_medial_joint: limit lower=0.0 upper=1.57 effort=20 velocity=2 -> lower=-0.05 upper=1.57 effort=30 velocity=4
- joint l_middle_proximal_joint: limit lower=0.0 upper=1.57 effort=20 velocity=2 -> lower=-0.05 upper=1.57 effort=30 velocity=4
- joint l_ring_distal_joint: limit lower=0.0 upper=1.0 effort=20 velocity=2 -> lower=-0.05 upper=1.0 effort=30 velocity=4
- joint l_ring_medial_joint: limit lower=0.0 upper=1.57 effort=20 velocity=2 -> lower=-0.05 upper=1.57 effort=30 velocity=4
- joint l_ring_proximal_joint: limit lower=0.0 upper=1.57 effort=20 velocity=2 -> lower=-0.05 upper=1.57 effort=30 velocity=4
- joint l_thumb_abduction_joint: limit lower=-0.6 upper=0.7853981633974483 effort=20 velocity=2 -> lower=-0.6 upper=0.7853981633974483 effort=30 velocity=4
- joint l_thumb_distal_joint: limit lower=0.0 upper=0.4 effort=20 velocity=2 -> lower=-0.05 upper=0.4 effort=30 velocity=4
- joint l_thumb_medial_joint: limit lower=0.0 upper=1.57 effort=20 velocity=2 -> lower=-0.05 upper=1.57 effort=30 velocity=4
- joint l_thumb_proximal_joint: limit lower=0.0 upper=0.8 effort=20 velocity=2 -> lower=-0.05 upper=0.8 effort=30 velocity=4
- joint l_wrist_adduction_joint: limit lower=-0.7853981633974483 upper=0.7853981633974483 effort=20 velocity=2 -> lower=-0.7853981633974483 upper=0.7853981633974483 effort=30 velocity=3
- joint l_wrist_flexion_joint: limit lower=-0.7853981633974483 upper=0.7853981633974483 effort=20 velocity=2 -> lower=-0.7853981633974483 upper=0.7853981633974483 effort=30 velocity=3
- joint l_wrist_rotation_joint: limit lower=-1.5707963267948966 upper=1.5707963267948966 effort=0.5 velocity=1.0 -> lower=-1.5707963267948966 upper=1.5707963267948966 effort=10 velocity=3

File: urdf/rh8d_macro.xacro (robot description, xacro)
@@ -27,5 +27,5 @@
       <child link="${prefix}forearm"/>
       <axis xyz="0 0 1"/>
-      <limit effort="0.5" lower="${-pi/2}" upper="${pi/2}" velocity="1.0"/>
+      <limit effort="10" lower="${-pi/2}" upper="${pi/2}" velocity="3"/>
     </joint>
     <link name="${prefix}forearm">
@@ -60,6 +60,6 @@
       <child link="${prefix}palm_axis"/>
       <axis xyz="0 0 1"/>
-      <limit effort="20" lower="${-pi/4}" upper="${pi/4}" velocity="2"/>
-      <dynamics damping="5" friction="0.0"/>
+      <limit effort="30" lower="${-pi/4}" upper="${pi/4}" velocity="3"/>
+      <dynamics damping="1" friction="0.0"/>
     </joint>
     <link name="${prefix}palm_axis">
@@ -82,6 +82,6 @@
       <child link="${prefix}palm"/>
       <axis xyz="0 0 1"/>
-      <limit effort="20" lower="${-pi/4}" upper="${pi/4}" velocity="2"/>
-      <dynamics damping="5" friction="0.0"/>
+      <limit effort="30" lower="${-pi/4}" upper="${pi/4}" velocity="3"/>
+      <dynamics damping="1" friction="0.0"/>
     </joint>
     <link name="${prefix}palm">

File: urdf/rh8d_right.urdf (robot description, URDF)
Before this commit: robot rh8d, 27 links, 26 joints
Joints:
- joint r_index_distal_joint: limit lower=0.0 upper=1.0 effort=20 velocity=2 -> lower=-0.05 upper=1.0 effort=30 velocity=4
- joint r_index_medial_joint: limit lower=0.0 upper=1.57 effort=20 velocity=2 -> lower=-0.05 upper=1.57 effort=30 velocity=4
- joint r_index_proximal_joint: limit lower=0.0 upper=1.57 effort=20 velocity=2 -> lower=-0.05 upper=1.57 effort=30 velocity=4
- joint r_little_distal_joint: limit lower=0.0 upper=1.0 effort=20 velocity=2 -> lower=-0.05 upper=1.0 effort=30 velocity=4
- joint r_little_medial_joint: limit lower=0.0 upper=1.57 effort=20 velocity=2 -> lower=-0.05 upper=1.57 effort=30 velocity=4
- joint r_little_proximal_joint: limit lower=0.0 upper=1.57 effort=20 velocity=2 -> lower=-0.05 upper=1.57 effort=30 velocity=4
- joint r_middle_distal_joint: limit lower=0.0 upper=1.0 effort=20 velocity=2 -> lower=-0.05 upper=1.0 effort=30 velocity=4
- joint r_middle_medial_joint: limit lower=0.0 upper=1.57 effort=20 velocity=2 -> lower=-0.05 upper=1.57 effort=30 velocity=4
- joint r_middle_proximal_joint: limit lower=0.0 upper=1.57 effort=20 velocity=2 -> lower=-0.05 upper=1.57 effort=30 velocity=4
- joint r_ring_distal_joint: limit lower=0.0 upper=1.0 effort=20 velocity=2 -> lower=-0.05 upper=1.0 effort=30 velocity=4
- joint r_ring_medial_joint: limit lower=0.0 upper=1.57 effort=20 velocity=2 -> lower=-0.05 upper=1.57 effort=30 velocity=4
- joint r_ring_proximal_joint: limit lower=0.0 upper=1.57 effort=20 velocity=2 -> lower=-0.05 upper=1.57 effort=30 velocity=4
- joint r_thumb_abduction_joint: limit lower=-0.6 upper=0.7853981633974483 effort=20 velocity=2 -> lower=-0.6 upper=0.7853981633974483 effort=30 velocity=4
- joint r_thumb_distal_joint: limit lower=0.0 upper=0.4 effort=20 velocity=2 -> lower=-0.05 upper=0.4 effort=30 velocity=4
- joint r_thumb_medial_joint: limit lower=0.0 upper=1.57 effort=20 velocity=2 -> lower=-0.05 upper=1.57 effort=30 velocity=4
- joint r_thumb_proximal_joint: limit lower=0.0 upper=0.8 effort=20 velocity=2 -> lower=-0.05 upper=0.8 effort=30 velocity=4
- joint r_wrist_adduction_joint: limit lower=-0.7853981633974483 upper=0.7853981633974483 effort=20 velocity=2 -> lower=-0.7853981633974483 upper=0.7853981633974483 effort=30 velocity=3
- joint r_wrist_flexion_joint: limit lower=-0.7853981633974483 upper=0.7853981633974483 effort=20 velocity=2 -> lower=-0.7853981633974483 upper=0.7853981633974483 effort=30 velocity=3
- joint r_wrist_rotation_joint: limit lower=-1.5707963267948966 upper=1.5707963267948966 effort=0.5 velocity=1.0 -> lower=-1.5707963267948966 upper=1.5707963267948966 effort=10 velocity=3
