Commit message: Double actuation speed (4x actual step response)
- Joint velocity limits doubled: phalanges 4->8 rad/s, wrist 3->6 rad/s.
- The real bottleneck was the control chain, not the limits:
  gz_ros2_control position_proportional_gain 0.1->0.3 (velocity command =
  gain * error * update_rate) and coupling-node trajectory horizon
  0.15->0.08 s.
- Measured: thumb step to 90% in 0.40 s (was 1.55), full sequential finger
  close in 0.40 s (was 1.60) at peak 8.0 rad/s = the limit. Overlap-sphere
  stability test still clean (no violations, settles to rest).

Co-Authored-By: Claude Fable 5 <noreply@anthropic.com>

File: urdf/rh8d.urdf.xacro (robot description, xacro)
@@ -58,4 +58,7 @@
         <plugin filename="gz_ros2_control-system" name="gz_ros2_control::GazeboSimROS2ControlPlugin">
           <parameters>$(arg controllers_file)</parameters>
+          <!-- velocity command = gain * position error * update_rate; the
+               default 0.1 caps joint speeds well below the URDF limits -->
+          <position_proportional_gain>0.3</position_proportional_gain>
         </plugin>
       </gazebo>

File: urdf/rh8d_finger.xacro (robot description, xacro)
@@ -14,5 +14,5 @@
        sticking against the palm until jostled). -->
   <xacro:property name="phalanx_effort"    value="30"/>
-  <xacro:property name="phalanx_velocity"  value="4"/>
+  <xacro:property name="phalanx_velocity"  value="8"/>
   <!-- Slightly negative lower limit: joints parked exactly ON a limit get
        pinned by dartsim's limit constraint and never move (frozen-thumb bug);

File: urdf/rh8d_left.urdf (robot description, URDF)
Before this commit: robot rh8d, 27 links, 26 joints
Joints:
- joint l_index_distal_joint: limit lower=-0.05 upper=1.0 effort=30 velocity=4 -> lower=-0.05 upper=1.0 effort=30 velocity=8
- joint l_index_medial_joint: limit lower=-0.05 upper=1.57 effort=30 velocity=4 -> lower=-0.05 upper=1.57 effort=30 velocity=8
- joint l_index_proximal_joint: limit lower=-0.05 upper=1.57 effort=30 velocity=4 -> lower=-0.05 upper=1.57 effort=30 velocity=8
- joint l_little_distal_joint: limit lower=-0.05 upper=1.0 effort=30 velocity=4 -> lower=-0.05 upper=1.0 effort=30 velocity=8
- joint l_little_medial_joint: limit lower=-0.05 upper=1.57 effort=30 velocity=4 -> lower=-0.05 upper=1.57 effort=30 velocity=8
- joint l_little_proximal_joint: limit lower=-0.05 upper=1.57 effort=30 velocity=4 -> lower=-0.05 upper=1.57 effort=30 velocity=8
- joint l_middle_distal_joint: limit lower=-0.05 upper=1.0 effort=30 velocity=4 -> lower=-0.05 upper=1.0 effort=30 velocity=8
- joint l_middle_medial_joint: limit lower=-0.05 upper=1.57 effort=30 velocity=4 -> lower=-0.05 upper=1.57 effort=30 velocity=8
- joint l_middle_proximal_joint: limit lower=-0.05 upper=1.57 effort=30 velocity=4 -> lower=-0.05 upper=1.57 effort=30 velocity=8
- joint l_ring_distal_joint: limit lower=-0.05 upper=1.0 effort=30 velocity=4 -> lower=-0.05 upper=1.0 effort=30 velocity=8
- joint l_ring_medial_joint: limit lower=-0.05 upper=1.57 effort=30 velocity=4 -> lower=-0.05 upper=1.57 effort=30 velocity=8
- joint l_ring_proximal_joint: limit lower=-0.05 upper=1.57 effort=30 velocity=4 -> lower=-0.05 upper=1.57 effort=30 velocity=8
- joint l_thumb_abduction_joint: limit lower=-0.6 upper=0.7853981633974483 effort=30 velocity=4 -> lower=-0.6 upper=0.7853981633974483 effort=30 velocity=8
- joint l_thumb_distal_joint: limit lower=-0.05 upper=0.4 effort=30 velocity=4 -> lower=-0.05 upper=0.4 effort=30 velocity=8
- joint l_thumb_medial_joint: limit lower=-0.05 upper=1.57 effort=30 velocity=4 -> lower=-0.05 upper=1.57 effort=30 velocity=8
- joint l_thumb_proximal_joint: limit lower=-0.05 upper=0.8 effort=30 velocity=4 -> lower=-0.05 upper=0.8 effort=30 velocity=8
- joint l_wrist_adduction_joint: limit lower=-0.7853981633974483 upper=0.7853981633974483 effort=30 velocity=3 -> lower=-0.7853981633974483 upper=0.7853981633974483 effort=30 velocity=6
- joint l_wrist_flexion_joint: limit lower=-0.7853981633974483 upper=0.7853981633974483 effort=30 velocity=3 -> lower=-0.7853981633974483 upper=0.7853981633974483 effort=30 velocity=6
- joint l_wrist_rotation_joint: limit lower=-1.5707963267948966 upper=1.5707963267948966 effort=10 velocity=3 -> lower=-1.5707963267948966 upper=1.5707963267948966 effort=10 velocity=6

File: urdf/rh8d_macro.xacro (robot description, xacro)
@@ -27,5 +27,5 @@
       <child link="${prefix}forearm"/>
       <axis xyz="0 0 1"/>
-      <limit effort="10" lower="${-pi/2}" upper="${pi/2}" velocity="3"/>
+      <limit effort="10" lower="${-pi/2}" upper="${pi/2}" velocity="6"/>
     </joint>
     <link name="${prefix}forearm">
@@ -60,5 +60,5 @@
       <child link="${prefix}palm_axis"/>
       <axis xyz="0 0 1"/>
-      <limit effort="30" lower="${-pi/4}" upper="${pi/4}" velocity="3"/>
+      <limit effort="30" lower="${-pi/4}" upper="${pi/4}" velocity="6"/>
       <dynamics damping="1" friction="0.0"/>
     </joint>
@@ -82,5 +82,5 @@
       <child link="${prefix}palm"/>
       <axis xyz="0 0 1"/>
-      <limit effort="30" lower="${-pi/4}" upper="${pi/4}" velocity="3"/>
+      <limit effort="30" lower="${-pi/4}" upper="${pi/4}" velocity="6"/>
       <dynamics damping="1" friction="0.0"/>
     </joint>

File: urdf/rh8d_right.urdf (robot description, URDF)
Before this commit: robot rh8d, 27 links, 26 joints
Joints:
- joint r_index_distal_joint: limit lower=-0.05 upper=1.0 effort=30 velocity=4 -> lower=-0.05 upper=1.0 effort=30 velocity=8
- joint r_index_medial_joint: limit lower=-0.05 upper=1.57 effort=30 velocity=4 -> lower=-0.05 upper=1.57 effort=30 velocity=8
- joint r_index_proximal_joint: limit lower=-0.05 upper=1.57 effort=30 velocity=4 -> lower=-0.05 upper=1.57 effort=30 velocity=8
- joint r_little_distal_joint: limit lower=-0.05 upper=1.0 effort=30 velocity=4 -> lower=-0.05 upper=1.0 effort=30 velocity=8
- joint r_little_medial_joint: limit lower=-0.05 upper=1.57 effort=30 velocity=4 -> lower=-0.05 upper=1.57 effort=30 velocity=8
- joint r_little_proximal_joint: limit lower=-0.05 upper=1.57 effort=30 velocity=4 -> lower=-0.05 upper=1.57 effort=30 velocity=8
- joint r_middle_distal_joint: limit lower=-0.05 upper=1.0 effort=30 velocity=4 -> lower=-0.05 upper=1.0 effort=30 velocity=8
- joint r_middle_medial_joint: limit lower=-0.05 upper=1.57 effort=30 velocity=4 -> lower=-0.05 upper=1.57 effort=30 velocity=8
- joint r_middle_proximal_joint: limit lower=-0.05 upper=1.57 effort=30 velocity=4 -> lower=-0.05 upper=1.57 effort=30 velocity=8
- joint r_ring_distal_joint: limit lower=-0.05 upper=1.0 effort=30 velocity=4 -> lower=-0.05 upper=1.0 effort=30 velocity=8
- joint r_ring_medial_joint: limit lower=-0.05 upper=1.57 effort=30 velocity=4 -> lower=-0.05 upper=1.57 effort=30 velocity=8
- joint r_ring_proximal_joint: limit lower=-0.05 upper=1.57 effort=30 velocity=4 -> lower=-0.05 upper=1.57 effort=30 velocity=8
- joint r_thumb_abduction_joint: limit lower=-0.6 upper=0.7853981633974483 effort=30 velocity=4 -> lower=-0.6 upper=0.7853981633974483 effort=30 velocity=8
- joint r_thumb_distal_joint: limit lower=-0.05 upper=0.4 effort=30 velocity=4 -> lower=-0.05 upper=0.4 effort=30 velocity=8
- joint r_thumb_medial_joint: limit lower=-0.05 upper=1.57 effort=30 velocity=4 -> lower=-0.05 upper=1.57 effort=30 velocity=8
- joint r_thumb_proximal_joint: limit lower=-0.05 upper=0.8 effort=30 velocity=4 -> lower=-0.05 upper=0.8 effort=30 velocity=8
- joint r_wrist_adduction_joint: limit lower=-0.7853981633974483 upper=0.7853981633974483 effort=30 velocity=3 -> lower=-0.7853981633974483 upper=0.7853981633974483 effort=30 velocity=6
- joint r_wrist_flexion_joint: limit lower=-0.7853981633974483 upper=0.7853981633974483 effort=30 velocity=3 -> lower=-0.7853981633974483 upper=0.7853981633974483 effort=30 velocity=6
- joint r_wrist_rotation_joint: limit lower=-1.5707963267948966 upper=1.5707963267948966 effort=10 velocity=3 -> lower=-1.5707963267948966 upper=1.5707963267948966 effort=10 velocity=6
