Commit message: Rename rh8d_description -> seed_rh8d_description
Adopt the seed_<scope>_<role> naming scheme. Updates the package/project
name, mesh URIs, xacro $(find) includes, launch files, test script, and
docs. Generated plain URDFs updated in place (URI-only change, no
regeneration needed).

Co-Authored-By: Claude Fable 5 <noreply@anthropic.com>

File: src/seed_rh8d_description/urdf/rh8d.urdf.xacro (robot description, xacro)
@@ -15,8 +15,8 @@
   <xacro:arg name="hardware_plugin" default="mock_components/GenericSystem"/>
   <xacro:arg name="controllers_file"
-             default="$(find rh8d_description)/config/rh8d_controllers_$(arg side).yaml"/>
-  <xacro:include filename="$(find rh8d_description)/urdf/rh8d_macro.xacro"/>
-  <xacro:include filename="$(find rh8d_description)/urdf/rh8d.gazebo.xacro"/>
-  <xacro:include filename="$(find rh8d_description)/urdf/rh8d.ros2_control.xacro"/>
+             default="$(find seed_rh8d_description)/config/rh8d_controllers_$(arg side).yaml"/>
+  <xacro:include filename="$(find seed_rh8d_description)/urdf/rh8d_macro.xacro"/>
+  <xacro:include filename="$(find seed_rh8d_description)/urdf/rh8d.gazebo.xacro"/>
+  <xacro:include filename="$(find seed_rh8d_description)/urdf/rh8d.ros2_control.xacro"/>
   <xacro:property name="side"   value="$(arg side)"/>
   <xacro:property name="prefix" value="${'l_' if side == 'left' else 'r_'}"/>

File: src/seed_rh8d_description/urdf/rh8d_finger.xacro (robot description, xacro)
@@ -30,5 +30,5 @@
         <origin rpy="0 0 0" xyz="0 0 0"/>
         <geometry>
-          <mesh filename="package://rh8d_description/meshes/phalanx_refac.stl" scale="0.001 0.001 0.001"/>
+          <mesh filename="package://seed_rh8d_description/meshes/phalanx_refac.stl" scale="0.001 0.001 0.001"/>
         </geometry>
         <material name="rh8d_black"/>
@@ -58,12 +58,12 @@
         <origin rpy="0 0 0" xyz="0 0 0"/>
         <geometry>
-          <mesh filename="package://rh8d_description/meshes/high_res/tip_refac.stl" scale="0.001 0.001 0.001"/>
-        </geometry>
-        <material name="rh8d_black"/>
-      </visual>
-      <collision>
-        <origin rpy="0 0 0" xyz="0 0 0"/>
-        <geometry>
-          <mesh filename="package://rh8d_description/meshes/tip_refac.stl" scale="0.001 0.001 0.001"/>
+          <mesh filename="package://seed_rh8d_description/meshes/high_res/tip_refac.stl" scale="0.001 0.001 0.001"/>
+        </geometry>
+        <material name="rh8d_black"/>
+      </visual>
+      <collision>
+        <origin rpy="0 0 0" xyz="0 0 0"/>
+        <geometry>
+          <mesh filename="package://seed_rh8d_description/meshes/tip_refac.stl" scale="0.001 0.001 0.001"/>
         </geometry>
       </collision>
@@ -88,5 +88,5 @@
         <origin rpy="0 0 0" xyz="0 0 0"/>
         <geometry>
-          <mesh filename="package://rh8d_description/meshes/high_res/sensor_refac.stl" scale="0.001 0.001 0.001"/>
+          <mesh filename="package://seed_rh8d_description/meshes/high_res/sensor_refac.stl" scale="0.001 0.001 0.001"/>
         </geometry>
         <material name="rh8d_sensor_green"/>
@@ -95,5 +95,5 @@
         <origin rpy="0 0 0" xyz="0 0 0"/>
         <geometry>
-          <mesh filename="package://rh8d_description/meshes/sensor_refac.stl" scale="0.001 0.001 0.001"/>
+          <mesh filename="package://seed_rh8d_description/meshes/sensor_refac.stl" scale="0.001 0.001 0.001"/>
         </geometry>
       </collision>
@@ -183,5 +183,5 @@
         <origin rpy="0 0 0" xyz="0 0 0"/>
         <geometry>
-          <mesh filename="package://rh8d_description/meshes/thumb_base_refac.stl" scale="0.001 0.001 0.001"/>
+          <mesh filename="package://seed_rh8d_description/meshes/thumb_base_refac.stl" scale="0.001 0.001 0.001"/>
         </geometry>
         <material name="rh8d_black"/>
@@ -205,5 +205,5 @@
         <origin rpy="0 0 0" xyz="0 0 0"/>
         <geometry>
-          <mesh filename="package://rh8d_description/meshes/thumb_phalanx_refac.stl" scale="0.001 0.001 0.001"/>
+          <mesh filename="package://seed_rh8d_description/meshes/thumb_phalanx_refac.stl" scale="0.001 0.001 0.001"/>
         </geometry>
         <material name="rh8d_black"/>
@@ -230,5 +230,5 @@
         <origin rpy="0 0 0" xyz="0 0 0"/>
         <geometry>
-          <mesh filename="package://rh8d_description/meshes/thumb_phalanx_refac.stl" scale="0.001 0.001 0.001"/>
+          <mesh filename="package://seed_rh8d_description/meshes/thumb_phalanx_refac.stl" scale="0.001 0.001 0.001"/>
         </geometry>
         <material name="rh8d_black"/>

File: src/seed_rh8d_description/urdf/rh8d_left.urdf (robot description, URDF)
Before this commit: robot rh8d, 27 links, 26 joints
Links:
- link l_forearm: geometry collision cylinder length=0.019 radius=0.025; collision mesh filename=package://seed_rh8d_description/meshes/forearm_collision.stl scale=0.001 0.001 0.001
- link l_index_distal: geometry collision mesh filename=package://seed_rh8d_description/meshes/tip_refac.stl scale=0.001 0.001 0.001; visual mesh filename=package://seed_rh8d_description/meshes/high_res/tip_refac.s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 scale=0.001 0.001 0.001
- link l_index_fingertip: geometry collision mesh filename=package://seed_rh8d_description/meshes/sensor_refac.stl scale=0.001 0.001 0.001; visual mesh filename=package://seed_rh8d_description/meshes/high_res/sensor_refa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 scale=0.001 0.001 0.001
- link l_index_medial: geometry collision cylinder length=0.0162 radius=0.008; collision sphere radius=0.008
- link l_index_proximal: geometry collision cylinder length=0.0162 radius=0.008; collision sphere radius=0.008
- link l_little_distal: geometry collision mesh filename=package://seed_rh8d_description/meshes/tip_refac.stl scale=0.001 0.001 0.001; visual mesh filename=package://seed_rh8d_description/meshes/high_res/tip_refac.s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 scale=0.001 0.001 0.001
- link l_little_fingertip: geometry collision mesh filename=package://seed_rh8d_description/meshes/sensor_refac.stl scale=0.001 0.001 0.001; visual mesh filename=package://seed_rh8d_description/meshes/high_res/sensor_refa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 scale=0.001 0.001 0.001
- link l_little_medial: geometry collision cylinder length=0.0162 radius=0.008; collision sphere radius=0.008
- link l_little_proximal: geometry collision cylinder length=0.0162 radius=0.008; collision sphere radius=0.008
- link l_middle_distal: geometry collision mesh filename=package://seed_rh8d_description/meshes/tip_refac.stl scale=0.001 0.001 0.001; visual mesh filename=package://seed_rh8d_description/meshes/high_res/tip_refac.s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 scale=0.001 0.001 0.001
- link l_middle_fingertip: geometry collision mesh filename=package://seed_rh8d_description/meshes/sensor_refac.stl scale=0.001 0.001 0.001; visual mesh filename=package://seed_rh8d_description/meshes/high_res/sensor_refa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 scale=0.001 0.001 0.001
- link l_middle_medial: geometry collision cylinder length=0.0162 radius=0.008; collision sphere radius=0.008
- link l_middle_proximal: geometry collision cylinder length=0.0162 radius=0.008; collision sphere radius=0.008
- link l_palm: geometry collision mesh filename=package://seed_rh8d_description/meshes/left_palm_collision.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 scale=0.001 0.001 0.001; visual mesh filename=package://seed_rh8d_description/meshes/high_res/left_palm_r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 scale=0.001 0.001 0.001
- link l_palm_axis: geometry visual mesh filename=package://seed_rh8d_description/meshes/palm_axis_refac.stl scale=0.001 0.001 0.001
- link l_ring_distal: geometry collision mesh filename=package://seed_rh8d_description/meshes/tip_refac.stl scale=0.001 0.001 0.001; visual mesh filename=package://seed_rh8d_description/meshes/high_res/tip_refac.s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 scale=0.001 0.001 0.001
- link l_ring_fingertip: geometry collision mesh filename=package://seed_rh8d_description/meshes/sensor_refac.stl scale=0.001 0.001 0.001; visual mesh filename=package://seed_rh8d_description/meshes/high_res/sensor_refa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 scale=0.001 0.001 0.001
- link l_ring_medial: geometry collision cylinder length=0.0162 radius=0.008; collision sphere radius=0.008
- link l_ring_proximal: geometry collision cylinder length=0.0162 radius=0.008; collision sphere radius=0.008
- link l_thumb_base: geometry visual mesh filename=package://seed_rh8d_description/meshes/thumb_base_refac.stl scale=0.001 0.001 0.001
- link l_thumb_distal: geometry collision mesh filename=package://seed_rh8d_description/meshes/tip_refac.stl scale=0.001 0.001 0.001; visual mesh filename=package://seed_rh8d_description/meshes/high_res/tip_refac.s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 scale=0.001 0.001 0.001
- link l_thumb_fingertip: geometry collision mesh filename=package://seed_rh8d_description/meshes/sensor_refac.stl scale=0.001 0.001 0.001; visual mesh filename=package://seed_rh8d_description/meshes/high_res/sensor_refa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 scale=0.001 0.001 0.001
- link l_thumb_medial: geometry collision cylinder length=0.011 radius=0.0074; collision sphere radius=0.0074
- link l_thumb_proximal: geometry visual mesh filename=package://seed_rh8d_description/meshes/thumb_phalanx_refac.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 scale=0.001 0.001 0.001

File: src/seed_rh8d_description/urdf/rh8d_macro.xacro (robot description, xacro)
@@ -1,6 +1,6 @@
 <?xml version="1.0"?>
 <robot xmlns:xacro="http://www.ros.org/wiki/xacro">
-  <xacro:include filename="$(find rh8d_description)/urdf/rh8d_materials.xacro"/>
-  <xacro:include filename="$(find rh8d_description)/urdf/rh8d_finger.xacro"/>
+  <xacro:include filename="$(find seed_rh8d_description)/urdf/rh8d_materials.xacro"/>
+  <xacro:include filename="$(find seed_rh8d_description)/urdf/rh8d_finger.xacro"/>
   <!--
     Seed Robotics RH8D hand.
@@ -38,5 +38,5 @@
         <origin rpy="0 0 0" xyz="0 0 0"/>
         <geometry>
-          <mesh filename="package://rh8d_description/meshes/forearm.stl" scale="0.001 0.001 0.001"/>
+          <mesh filename="package://seed_rh8d_description/meshes/forearm.stl" scale="0.001 0.001 0.001"/>
         </geometry>
         <material name="rh8d_black"/>
@@ -51,5 +51,5 @@
         <origin rpy="0 0 0" xyz="0 0 0"/>
         <geometry>
-          <mesh filename="package://rh8d_description/meshes/forearm_collision.stl" scale="0.001 0.001 0.001"/>
+          <mesh filename="package://seed_rh8d_description/meshes/forearm_collision.stl" scale="0.001 0.001 0.001"/>
         </geometry>
       </collision>
@@ -72,5 +72,5 @@
         <origin rpy="0 0 0" xyz="0 0 0"/>
         <geometry>
-          <mesh filename="package://rh8d_description/meshes/palm_axis_refac.stl" scale="0.001 0.001 0.001"/>
+          <mesh filename="package://seed_rh8d_description/meshes/palm_axis_refac.stl" scale="0.001 0.001 0.001"/>
         </geometry>
         <material name="rh8d_black"/>
@@ -94,5 +94,5 @@
         <origin rpy="0 0 0" xyz="0 0 0"/>
         <geometry>
-          <mesh filename="package://rh8d_description/meshes/high_res/${side}_palm_refac.stl" scale="0.001 0.001 0.001"/>
+          <mesh filename="package://seed_rh8d_description/meshes/high_res/${side}_palm_refac.stl" scale="0.001 0.001 0.001"/>
         </geometry>
         <material name="rh8d_black"/>
@@ -101,5 +101,5 @@
         <origin rpy="0 0 0" xyz="0 0 0"/>
         <geometry>
-          <mesh filename="package://rh8d_description/meshes/${side}_palm_collision.stl" scale="0.001 0.001 0.001"/>
+          <mesh filename="package://seed_rh8d_description/meshes/${side}_palm_collision.stl" scale="0.001 0.001 0.001"/>
         </geometry>
       </collision>

File: src/seed_rh8d_description/urdf/rh8d_right.urdf (robot description, URDF)
Before this commit: robot rh8d, 27 links, 26 joints
Links:
- link r_forearm: geometry collision cylinder length=0.019 radius=0.025; collision mesh filename=package://seed_rh8d_description/meshes/forearm_collision.stl scale=0.001 0.001 0.001
- link r_index_distal: geometry collision mesh filename=package://seed_rh8d_description/meshes/tip_refac.stl scale=0.001 0.001 0.001; visual mesh filename=package://seed_rh8d_description/meshes/high_res/tip_refac.s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 scale=0.001 0.001 0.001
- link r_index_fingertip: geometry collision mesh filename=package://seed_rh8d_description/meshes/sensor_refac.stl scale=0.001 0.001 0.001; visual mesh filename=package://seed_rh8d_description/meshes/high_res/sensor_refa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 scale=0.001 0.001 0.001
- link r_index_medial: geometry collision cylinder length=0.0162 radius=0.008; collision sphere radius=0.008
- link r_index_proximal: geometry collision cylinder length=0.0162 radius=0.008; collision sphere radius=0.008
- link r_little_distal: geometry collision mesh filename=package://seed_rh8d_description/meshes/tip_refac.stl scale=0.001 0.001 0.001; visual mesh filename=package://seed_rh8d_description/meshes/high_res/tip_refac.s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 scale=0.001 0.001 0.001
- link r_little_fingertip: geometry collision mesh filename=package://seed_rh8d_description/meshes/sensor_refac.stl scale=0.001 0.001 0.001; visual mesh filename=package://seed_rh8d_description/meshes/high_res/sensor_refa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 scale=0.001 0.001 0.001
- link r_little_medial: geometry collision cylinder length=0.0162 radius=0.008; collision sphere radius=0.008
- link r_little_proximal: geometry collision cylinder length=0.0162 radius=0.008; collision sphere radius=0.008
- link r_middle_distal: geometry collision mesh filename=package://seed_rh8d_description/meshes/tip_refac.stl scale=0.001 0.001 0.001; visual mesh filename=package://seed_rh8d_description/meshes/high_res/tip_refac.s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 scale=0.001 0.001 0.001
- link r_middle_fingertip: geometry collision mesh filename=package://seed_rh8d_description/meshes/sensor_refac.stl scale=0.001 0.001 0.001; visual mesh filename=package://seed_rh8d_description/meshes/high_res/sensor_refa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 scale=0.001 0.001 0.001
- link r_middle_medial: geometry collision cylinder length=0.0162 radius=0.008; collision sphere radius=0.008
- link r_middle_proximal: geometry collision cylinder length=0.0162 radius=0.008; collision sphere radius=0.008
- link r_palm: geometry collision mesh filename=package://seed_rh8d_description/meshes/right_palm_collision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 scale=0.001 0.001 0.001; visual mesh filename=package://seed_rh8d_description/meshes/high_res/right_palm_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 scale=0.001 0.001 0.001
- link r_palm_axis: geometry visual mesh filename=package://seed_rh8d_description/meshes/palm_axis_refac.stl scale=0.001 0.001 0.001
- link r_ring_distal: geometry collision mesh filename=package://seed_rh8d_description/meshes/tip_refac.stl scale=0.001 0.001 0.001; visual mesh filename=package://seed_rh8d_description/meshes/high_res/tip_refac.s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 scale=0.001 0.001 0.001
- link r_ring_fingertip: geometry collision mesh filename=package://seed_rh8d_description/meshes/sensor_refac.stl scale=0.001 0.001 0.001; visual mesh filename=package://seed_rh8d_description/meshes/high_res/sensor_refa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 scale=0.001 0.001 0.001
- link r_ring_medial: geometry collision cylinder length=0.0162 radius=0.008; collision sphere radius=0.008
- link r_ring_proximal: geometry collision cylinder length=0.0162 radius=0.008; collision sphere radius=0.008
- link r_thumb_base: geometry visual mesh filename=package://seed_rh8d_description/meshes/thumb_base_refac.stl scale=0.001 0.001 0.001
- link r_thumb_distal: geometry collision mesh filename=package://seed_rh8d_description/meshes/tip_refac.stl scale=0.001 0.001 0.001; visual mesh filename=package://seed_rh8d_description/meshes/high_res/tip_refac.s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 scale=0.001 0.001 0.001
- link r_thumb_fingertip: geometry collision mesh filename=package://seed_rh8d_description/meshes/sensor_refac.stl scale=0.001 0.001 0.001; visual mesh filename=package://seed_rh8d_description/meshes/high_res/sensor_refa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 scale=0.001 0.001 0.001
- link r_thumb_medial: geometry collision cylinder length=0.011 radius=0.0074; collision sphere radius=0.0074
- link r_thumb_proximal: geometry visual mesh filename=package://seed_rh8d_description/meshes/thumb_phalanx_refac.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 scale=0.001 0.001 0.001
