Commit message: refactor and rokoko glove control added

File: src/seed_rh8d_description/urdf/rh8d.ros2_control.xacro (robot description, xacro)
@@ -46,5 +46,5 @@
       <xacro:rh8d_joint_iface joint="${prefix}wrist_adduction_joint"/>
       <xacro:rh8d_joint_iface joint="${prefix}wrist_flexion_joint"/>
-      <xacro:rh8d_joint_iface joint="${prefix}thumb_abduction_joint"/>
+      <xacro:rh8d_joint_iface joint="${prefix}thumb_adduction_joint"/>
       <xacro:if value="${finger_coupling == 'mimic'}">
         <xacro:rh8d_joint_iface joint="${prefix}thumb_proximal_joint"/>

File: src/seed_rh8d_description/urdf/rh8d_finger.xacro (robot description, xacro)
@@ -166,5 +166,5 @@
     <xacro:property name="prox_joint" value="${prefix}thumb_proximal_joint"/>
     <xacro:property name="mimic_base" value="${leader if leader != '' else prox_joint}"/>
-    <joint name="${prefix}thumb_abduction_joint" type="revolute">
+    <joint name="${prefix}thumb_adduction_joint" type="revolute">
       <origin rpy="${mount_rpy}" xyz="${mount_xyz}"/>
       <parent link="${prefix}palm"/>

File: src/seed_rh8d_description/urdf/rh8d_left.urdf (robot description, URDF)
Before this commit: robot rh8d, 27 links, 26 joints
Joints:
- removed joint l_thumb_abduction_joint
- added joint l_thumb_adduction_joint: type revolute, parent l_palm, child l_thumb_base, origin xyz=-0.0083412575 0.0157859987 -0.0379541955 rpy=0.60093862 -0.59510795 -2.8183247, axis 0 0 1, limit lower=-0.6 upper=0.7853981633974483 effort=30 velocity=8

File: src/seed_rh8d_description/urdf/rh8d_macro.xacro (robot description, xacro)
@@ -28,4 +28,8 @@
       <axis xyz="0 0 1"/>
       <limit effort="10" lower="${-pi/2}" upper="${pi/2}" velocity="6"/>
+      <!-- Without damping a large step command overshoots into the joint
+           limit, where dartsim pins the joint permanently (the other two
+           wrist axes have carried damping="1" from the start). -->
+      <dynamics damping="1" friction="0.0"/>
     </joint>
     <link name="${prefix}forearm">

File: src/seed_rh8d_description/urdf/rh8d_right.urdf (robot description, URDF)
Before this commit: robot rh8d, 27 links, 26 joints
Joints:
- removed joint r_thumb_abduction_joint
- added joint r_thumb_adduction_joint: type revolute, parent r_palm, child r_thumb_base, origin xyz=-0.0083412575 0.0157859987 0.0379541955 rpy=-2.54680616 -0.60124514 0.33418237, axis 0 0 -1, limit lower=-0.6 upper=0.7853981633974483 effort=30 velocity=8
