Commit message: added selfcollision

File: src/seed_rh8d_description/urdf/rh8d.gazebo.xacro (robot description, xacro)
@@ -50,4 +50,10 @@
       <plugin filename="gz-sim-joint-state-publisher-system"
               name="gz::sim::systems::JointStatePublisher"/>
+      <!-- Self-collision is a MODEL-level switch in gz-sim: the per-link
+           <self_collide> below is not what turns it on, and without this the
+           thumb sweeps straight through a closed fist. Links joined by a
+           joint are still exempt, so the phalanx chains do not fight their
+           own neighbours. -->
+      <self_collide>true</self_collide>
     </gazebo>
     <xacro:rh8d_link_friction link="${prefix}forearm"/>

File: src/seed_rh8d_description/urdf/rh8d_finger.xacro (robot description, xacro)
@@ -209,4 +209,14 @@
         <material name="rh8d_black"/>
       </visual>
+      <!-- Slimmer than thumb_medial's, and kept to the distal half of the
+           link: the thumb mount is calibrated per side rather than mirrored,
+           so a volume sized like the medial one clears the palm on the right
+           and sits inside it on the left, jamming the abduction axis. -->
+      <collision>
+        <origin rpy="${pi/2} 0 0" xyz="0 -0.015 0"/>
+        <geometry>
+          <cylinder length="0.010" radius="0.0050"/>
+        </geometry>
+      </collision>
     </link>
     <joint name="${prefix}thumb_medial_joint" type="revolute">
